Commit message: tmp branch

File: avatars/MetaHuman/urdf/avatar.urdf.xacro (robot description, xacro)
@@ -1,4 +1,7 @@
 <?xml version="1.0" encoding="UTF-8"?>
 <robot xmlns:xacro="http://ros.org/wiki/xacro" name="avatar">
+    <xacro:arg name="prefix" default="avatar/" />
+    <xacro:property name="avatar_prefix"
+                    value="$(arg prefix)"/>
     <xacro:property name="mesh_folder"
                     value="package://iai_avatar_description/avatars/MetaHuman/meshes/fbx"/>
@@ -22,176 +25,176 @@
     </xacro:macro>
     <xacro:macro name="yaw_pitch_joints" params="linkname mass">
-        <link name="${linkname}_yaw">
+        <link name="${avatar_prefix}${linkname}_yaw">
             <xacro:default_inertial mass="${mass}"/>
         </link>
-        <link name="${linkname}_pitch">
+        <link name="${avatar_prefix}${linkname}_pitch">
             <xacro:default_inertial mass="${mass}"/>
         </link>
     </xacro:macro>
-    <link name="root"/>
-    <link name="pelvis">
+    <link name="${avatar_prefix}root"/>
+    <link name="${avatar_prefix}pelvis">
         <xacro:mesh_coll bpart="pelvis"/>
         <xacro:default_inertial mass="8.36"/>
     </link>
     <xacro:yaw_pitch_joints linkname="pelvis" mass="8.36"/>
-    <link name="spine_01">
+    <link name="${avatar_prefix}spine_01">
         <xacro:default_inertial mass="2.34"/>
     </link>
-    <link name="spine_02">
+    <link name="${avatar_prefix}spine_02">
         <xacro:default_inertial mass="3.34"/>
     </link>
-    <link name="spine_03">
+    <link name="${avatar_prefix}spine_03">
         <xacro:default_inertial mass="4.43"/>
     </link>
-    <link name="spine_04">
+    <link name="${avatar_prefix}spine_04">
         <xacro:mesh_coll bpart="torso"/>
         <xacro:default_inertial mass="5.43"/>
     </link>
     <xacro:yaw_pitch_joints linkname="spine_04" mass="5.43"/>
-    <link name="spine_05">
+    <link name="${avatar_prefix}spine_05">
         <xacro:default_inertial mass="6.05"/>
     </link>
-    <link name="neck_01">
+    <link name="${avatar_prefix}neck_01">
         <xacro:default_inertial mass="1.39"/>
     </link>
-    <link name="neck_02">
+    <link name="${avatar_prefix}neck_02">
         <xacro:default_inertial mass="1.34"/>
     </link>
-    <link name="head">
+    <link name="${avatar_prefix}head">
         <xacro:mesh_coll bpart="head"/>
         <xacro:default_inertial mass="3.34"/>
     </link>
     <xacro:yaw_pitch_joints linkname="head" mass="3.34"/>
-    <link name="clavicle_l">
+    <link name="${avatar_prefix}clavicle_l">
         <xacro:default_inertial mass="2.08"/>
     </link>
-    <link name="upperarm_l">
+    <link name="${avatar_prefix}upperarm_l">
         <xacro:mesh_coll bpart="upperarm_l"/>
         <xacro:default_inertial mass="1.75"/>
     </link>
     <xacro:yaw_pitch_joints linkname="upperarm_l" mass="1.75"/>
-    <link name="lowerarm_l">
+    <link name="${avatar_prefix}lowerarm_l">
         <xacro:mesh_coll bpart="lowerarm_l"/>
         <xacro:default_inertial mass="1.39"/>
     </link>
     <xacro:yaw_pitch_joints linkname="lowerarm_l" mass="1.39"/>
-    <link name="hand_l">
+    <link name="${avatar_prefix}hand_l">
         <xacro:mesh_coll bpart="hand_l"/>
         <xacro:default_inertial mass="1.56"/>
     </link>
     <xacro:yaw_pitch_joints linkname="hand_l" mass="1.56"/>
-    <link name="clavicle_r">
+    <link name="${avatar_prefix}clavicle_r">
         <xacro:default_inertial mass="2.09"/>
     </link>
-    <link name="upperarm_r">
+    <link name="${avatar_prefix}upperarm_r">
         <xacro:mesh_coll bpart="upperarm_r"/>
         <xacro:default_inertial mass="1.75"/>
     </link>
     <xacro:yaw_pitch_joints linkname="upperarm_r" mass="1.75"/>
-    <link name="lowerarm_r">
+    <link name="${avatar_prefix}lowerarm_r">
         <xacro:mesh_coll bpart="lowerarm_r"/>
         <xacro:default_inertial mass="1.39"/>
     </link>
     <xacro:yaw_pitch_joints linkname="lowerarm_r" mass="1.39"/>
-    <link name="hand_r">
+    <link name="${avatar_prefix}hand_r">
         <xacro:mesh_coll bpart="hand_r"/>
         <xacro:default_inertial mass="1.15"/>
     </link>
     <xacro:yaw_pitch_joints linkname="hand_r" mass="1.15"/>
-    <link name="thigh_l">
+    <link name="${avatar_prefix}thigh_l">
         <xacro:mesh_coll bpart="thigh_l"/>
         <xacro:default_inertial mass="5.50"/>
     </link>
-    <link name="calf_l">
+    <link name="${avatar_prefix}calf_l">
         <xacro:mesh_coll bpart="calf_l"/>
         <xacro:default_inertial mass="3.37"/>
     </link>
-    <link name="foot_l">
+    <link name="${avatar_prefix}foot_l">
         <xacro:mesh_coll bpart="foot_l"/>
         <xacro:default_inertial mass="1.12"/>
     </link>
-    <link name="thigh_r">
+    <link name="${avatar_prefix}thigh_r">
         <xacro:mesh_coll bpart="thigh_r"/>
         <xacro:default_inertial mass="5.50"/>
     </link>
-    <link name="calf_r">
+    <link name="${avatar_prefix}calf_r">
         <xacro:mesh_coll bpart="calf_r"/>
         <xacro:default_inertial mass="3.37"/>
     </link>
-    <link name="foot_r">
+    <link name="${avatar_prefix}foot_r">
         <xacro:mesh_coll bpart="foot_r"/>
         <xacro:default_inertial mass="1.12"/>
     </link>
-    <joint name="root_to_pelvis_yaw" type="fixed">
-        <parent link="root"/>
-        <child link="pelvis_yaw"/>
+    <joint name="${avatar_prefix}root_to_${avatar_prefix}pelvis_yaw" type="fixed">
+        <parent link="${avatar_prefix}root"/>
+        <child link="${avatar_prefix}pelvis_yaw"/>
         <origin rpy="0 -1.5708 0" xyz="0 0 0.8854"/>
     </joint>
-    <joint name="pelvis_yaw_to_pelvis_pitch" type="revolute">
-        <parent link="pelvis_yaw"/>
-        <child link="pelvis_pitch"/>
-        <limit effort="1" lower="-1.5708" upper="2.44346" velocity="1"/>
-        <origin rpy="0 0 0" xyz="0 0 0"/>
-        <axis xyz="0 1 0"/>
-    </joint>
-    <joint name="pelvis_pitch_to_pelvis" type="revolute">
-        <parent link="pelvis_pitch"/>
-        <child link="pelvis"/>
-        <limit effort="1" lower="-1.5708" upper="2.44346" velocity="1"/>
-        <origin rpy="0 0 0" xyz="0 0 0"/>
-        <axis xyz="1 0 0"/>
-    </joint>
-    <joint name="pelvis_to_spine_01_yaw" type="revolute">
-        <parent link="pelvis"/>
-        <child link="spine_01"/>
+    <joint name="${avatar_prefix}pelvis_yaw_to_${avatar_prefix}pelvis_pitch" type="revolute">
+        <parent link="${avatar_prefix}pelvis_yaw"/>
+        <child link="${avatar_prefix}pelvis_pitch"/>
+        <limit effort="1" lower="-1.5708" upper="2.44346" velocity="1"/>
+        <origin rpy="0 0 0" xyz="0 0 0"/>
+        <axis xyz="0 1 0"/>
+    </joint>
+    <joint name="${avatar_prefix}pelvis_pitch_to_${avatar_prefix}pelvis" type="revolute">
+        <parent link="${avatar_prefix}pelvis_pitch"/>
+        <child link="${avatar_prefix}pelvis"/>
+        <limit effort="1" lower="-1.5708" upper="2.44346" velocity="1"/>
+        <origin rpy="0 0 0" xyz="0 0 0"/>
+        <axis xyz="1 0 0"/>
+    </joint>
+    <joint name="${avatar_prefix}pelvis_to_${avatar_prefix}spine_01_yaw" type="revolute">
+        <parent link="${avatar_prefix}pelvis"/>
+        <child link="${avatar_prefix}spine_01"/>
         <limit effort="1" lower="0" upper="0" velocity="1"/>
         <origin rpy="0 0 0" xyz="0.02031170 0 0"/>
         <axis xyz="1 0 0"/>
     </joint>
-    <joint name="spine_01_to_spine_02" type="continuous">
-        <parent link="spine_01"/>
-        <child link="spine_02"/>
+    <joint name="${avatar_prefix}spine_01_to_${avatar_prefix}spine_02" type="continuous">
+        <parent link="${avatar_prefix}spine_01"/>
+        <child link="${avatar_prefix}spine_02"/>
         <dynamics damping="1.0" friction="0.0001"/>
         <origin rpy="0 0 0" xyz="0.042 0 0"/>
         <axis xyz="1 0 0"/>
     </joint>
-    <joint name="spine_02_to_spine_03" type="revolute">
-        <parent link="spine_02"/>
-        <child link="spine_03"/>
+    <joint name="${avatar_prefix}spine_02_to_${avatar_prefix}spine_03" type="revolute">
+        <parent link="${avatar_prefix}spine_02"/>
+        <child link="${avatar_prefix}spine_03"/>
         <limit effort="1" lower="0" upper="0" velocity="1"/>
         <origin rpy="0 0 0" xyz="0.067 0 0"/>
         <axis xyz="1 0 0"/>
     </joint>
-    <joint name="spine_03_to_spine_04_yaw" type="revolute">
-        <parent link="spine_03"/>
-        <child link="spine_04_yaw"/>
+    <joint name="${avatar_prefix}spine_03_to_${avatar_prefix}spine_04_yaw" type="revolute">
+        <parent link="${avatar_prefix}spine_03"/>
+        <child link="${avatar_prefix}spine_04_yaw"/>
         <limit effort="1" lower="0" upper="0" velocity="1"/>
         <origin rpy="0 0 0" xyz="0.07891 0 0"/>
         <axis xyz="1 0 0"/>
     </joint>
-    <joint name="spine_04_yaw_to_spine_04_pitch" type="revolute">
-        <parent link="spine_04_yaw"/>
-        <child link="spine_04_pitch"/>
-        <limit effort="1" lower="-1.5708" upper="2.44346" velocity="1"/>
-        <origin rpy="0 0 0" xyz="0 0 0"/>
-        <axis xyz="0 1 0"/>
-    </joint>
-    <joint name="spine_04_pitch_to_spine_04" type="revolute">
-        <parent link="spine_04_pitch"/>
-        <child link="spine_04"/>
-        <limit effort="1" lower="-1.5708" upper="2.44346" velocity="1"/>
-        <origin rpy="0 0 0" xyz="0 0 0"/>
-        <axis xyz="1 0 0"/>
-    </joint>
-    <joint name="spine_04_to_spine_05" type="continuous">
-        <parent link="spine_04"/>
-        <child link="spine_05"/>
+    <joint name="${avatar_prefix}spine_04_yaw_to_${avatar_prefix}spine_04_pitch" type="revolute">
+        <parent link="${avatar_prefix}spine_04_yaw"/>
+        <child link="${avatar_prefix}spine_04_pitch"/>
+        <limit effort="1" lower="-1.5708" upper="2.44346" velocity="1"/>
+        <origin rpy="0 0 0" xyz="0 0 0"/>
+        <axis xyz="0 1 0"/>
+    </joint>
+    <joint name="${avatar_prefix}spine_04_pitch_to_${avatar_prefix}spine_04" type="revolute">
+        <parent link="${avatar_prefix}spine_04_pitch"/>
+        <child link="${avatar_prefix}spine_04"/>
+        <limit effort="1" lower="-1.5708" upper="2.44346" velocity="1"/>
+        <origin rpy="0 0 0" xyz="0 0 0"/>
+        <axis xyz="1 0 0"/>
+    </joint>
+    <joint name="${avatar_prefix}spine_04_to_${avatar_prefix}spine_05" type="continuous">
+        <parent link="${avatar_prefix}spine_04"/>
+        <child link="${avatar_prefix}spine_05"/>
         <dynamics damping="1.0" friction="0.0001"/>
         <origin rpy="0 0 0" xyz="0.15038425 0 0"/>
         <axis xyz="1 0 0"/>
     </joint>
-    <joint name="spine_05_to_neck_01" type="revolute">
-        <parent link="spine_05"/>
-        <child link="neck_01"/>
+    <joint name="${avatar_prefix}spine_05_to_${avatar_prefix}neck_01" type="revolute">
+        <parent link="${avatar_prefix}spine_05"/>
+        <child link="${avatar_prefix}neck_01"/>
         <dynamics damping="1.0" friction="0.0001"/>
         <limit effort="1" lower="-1.22173" upper="1.22173" velocity="1"/>
@@ -199,7 +202,7 @@
         <axis xyz="1 0 0"/>
     </joint>
-    <joint name="neck_01_to_neck_02" type="revolute">
-        <parent link="neck_01"/>
-        <child link="neck_02"/>
+    <joint name="${avatar_prefix}neck_01_to_${avatar_prefix}neck_02" type="revolute">
+        <parent link="${avatar_prefix}neck_01"/>
+        <child link="${avatar_prefix}neck_02"/>
         <dynamics damping="1.0" friction="0.0001"/>
         <limit effort="1" lower="-1.5708" upper="0.959931" velocity="1"/>
@@ -207,7 +210,7 @@
         <axis xyz="0 0 1"/>
     </joint>
-    <joint name="neck_02_to_head_yaw" type="revolute">
-        <parent link="neck_02"/>
-        <child link="head_yaw"/>
+    <joint name="${avatar_prefix}neck_02_to_${avatar_prefix}head_yaw" type="revolute">
+        <parent link="${avatar_prefix}neck_02"/>
+        <child link="${avatar_prefix}head_yaw"/>
         <dynamics damping="1.0" friction="0.0001"/>
         <limit effort="1" lower="-0.610865" upper="0.610865" velocity="1"/>
@@ -215,21 +218,21 @@
         <axis xyz="0 1 0"/>
     </joint>
-    <joint name="head_yaw_to_head_pitch" type="revolute">
-        <parent link="head_yaw"/>
-        <child link="head_pitch"/>
-        <limit effort="1" lower="-1.5708" upper="2.44346" velocity="1"/>
-        <origin rpy="0 0 0" xyz="0 0 0"/>
-        <axis xyz="0 1 0"/>
-    </joint>
-    <joint name="head_pitch_to_head" type="revolute">
-        <parent link="head_pitch"/>
-        <child link="head"/>
-        <limit effort="1" lower="-1.5708" upper="2.44346" velocity="1"/>
-        <origin rpy="0 0 0" xyz="0 0 0"/>
-        <axis xyz="1 0 0"/>
-    </joint>
-    <joint name="spine_05_to_clavicle_l" type="revolute">
-        <parent link="spine_05"/>
-        <child link="clavicle_l"/>
+    <joint name="${avatar_prefix}head_yaw_to_${avatar_prefix}head_pitch" type="revolute">
+        <parent link="${avatar_prefix}head_yaw"/>
+        <child link="${avatar_prefix}head_pitch"/>
+        <limit effort="1" lower="-1.5708" upper="2.44346" velocity="1"/>
+        <origin rpy="0 0 0" xyz="0 0 0"/>
+        <axis xyz="0 1 0"/>
+    </joint>
+    <joint name="${avatar_prefix}head_pitch_to_${avatar_prefix}head" type="revolute">
+        <parent link="${avatar_prefix}head_pitch"/>
+        <child link="${avatar_prefix}head"/>
+        <limit effort="1" lower="-1.5708" upper="2.44346" velocity="1"/>
+        <origin rpy="0 0 0" xyz="0 0 0"/>
+        <axis xyz="1 0 0"/>
+    </joint>
+    <joint name="${avatar_prefix}spine_05_to_${avatar_prefix}clavicle_l" type="revolute">
+        <parent link="${avatar_prefix}spine_05"/>
+        <child link="${avatar_prefix}clavicle_l"/>
         <origin rpy="0 1.5708 0" xyz="0.05142808 0.00883206 -0.00816548"/>
         <dynamics damping="1.0" friction="0.0001"/>
@@ -237,7 +240,7 @@
         <axis xyz="0 1 0"/>
     </joint>
-    <joint name="clavicle_l_to_upperarm_l_yaw" type="revolute">
-        <parent link="clavicle_l"/>
-        <child link="upperarm_l_yaw"/>
+    <joint name="${avatar_prefix}clavicle_l_to_${avatar_prefix}upperarm_l_yaw" type="revolute">
+        <parent link="${avatar_prefix}clavicle_l"/>
+        <child link="${avatar_prefix}upperarm_l_yaw"/>
         <dynamics damping="1.0" friction="0.0001"/>
         <limit effort="1" lower="-1.5708" upper="2.44346" velocity="1"/>
@@ -245,90 +248,90 @@
         <axis xyz="0 0 1"/>
     </joint>
-    <joint name="upperarm_l_yaw_to_upperarm_l_pitch" type="revolute">
-        <parent link="upperarm_l_yaw"/>
-        <child link="upperarm_l_pitch"/>
-        <limit effort="1" lower="-1.5708" upper="2.44346" velocity="1"/>
-        <origin rpy="0 0 0" xyz="0 0 0"/>
-        <axis xyz="0 1 0"/>
-    </joint>
-    <joint name="upperarm_l_pitch_to_upperarm_l" type="revolute">
-        <parent link="upperarm_l_pitch"/>
-        <child link="upperarm_l"/>
-        <limit effort="1" lower="-1.5708" upper="2.44346" velocity="1"/>
-        <origin rpy="0 0 0" xyz="0 0 0"/>
-        <axis xyz="1 0 0"/>
-    </joint>
-    <joint name="upperarm_l_to_lowerarm_l_yaw" type="continuous">
-        <parent link="upperarm_l"/>
-        <child link="lowerarm_l_yaw"/>
+    <joint name="${avatar_prefix}upperarm_l_yaw_to_${avatar_prefix}upperarm_l_pitch" type="revolute">
+        <parent link="${avatar_prefix}upperarm_l_yaw"/>
+        <child link="${avatar_prefix}upperarm_l_pitch"/>
+        <limit effort="1" lower="-1.5708" upper="2.44346" velocity="1"/>
+        <origin rpy="0 0 0" xyz="0 0 0"/>
+        <axis xyz="0 1 0"/>
+    </joint>
+    <joint name="${avatar_prefix}upperarm_l_pitch_to_${avatar_prefix}upperarm_l" type="revolute">
+        <parent link="${avatar_prefix}upperarm_l_pitch"/>
+        <child link="${avatar_prefix}upperarm_l"/>
+        <limit effort="1" lower="-1.5708" upper="2.44346" velocity="1"/>
+        <origin rpy="0 0 0" xyz="0 0 0"/>
+        <axis xyz="1 0 0"/>
+    </joint>
+    <joint name="${avatar_prefix}upperarm_l_to_${avatar_prefix}lowerarm_l_yaw" type="continuous">
+        <parent link="${avatar_prefix}upperarm_l"/>
+        <child link="${avatar_prefix}lowerarm_l_yaw"/>
         <origin rpy="0 0 0" xyz="0.238537997 0 0"/>
         <axis xyz="1 0 0"/>
     </joint>
-    <joint name="lowerarm_l_yaw_to_lowerarm_l_pitch" type="revolute">
-        <parent link="lowerarm_l_yaw"/>
-        <child link="lowerarm_l_pitch"/>
-        <limit effort="1" lower="-1.5708" upper="2.44346" velocity="1"/>
-        <origin rpy="0 0 0" xyz="0 0 0"/>
-        <axis xyz="0 1 0"/>
-    </joint>
-    <joint name="lowerarm_l_pitch_to_lowerarm_l" type="revolute">
-        <parent link="lowerarm_l_pitch"/>
-        <child link="lowerarm_l"/>
-        <limit effort="1" lower="-1.5708" upper="2.44346" velocity="1"/>
-        <origin rpy="0 0 0" xyz="0 0 0"/>
-        <axis xyz="1 0 0"/>
-    </joint>
-    <joint name="lowerarm_l_to_hand_l_yaw" type="continuous">
-        <parent link="lowerarm_l"/>
-        <child link="hand_l_yaw"/>
+    <joint name="${avatar_prefix}lowerarm_l_yaw_to_${avatar_prefix}lowerarm_l_pitch" type="revolute">
+        <parent link="${avatar_prefix}lowerarm_l_yaw"/>
+        <child link="${avatar_prefix}lowerarm_l_pitch"/>
+        <limit effort="1" lower="-1.5708" upper="2.44346" velocity="1"/>
+        <origin rpy="0 0 0" xyz="0 0 0"/>
+        <axis xyz="0 1 0"/>
+    </joint>
+    <joint name="${avatar_prefix}lowerarm_l_pitch_to_${avatar_prefix}lowerarm_l" type="revolute">
+        <parent link="${avatar_prefix}lowerarm_l_pitch"/>
+        <child link="${avatar_prefix}lowerarm_l"/>
+        <limit effort="1" lower="-1.5708" upper="2.44346" velocity="1"/>
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