Commit message: new joints for legs

File: avatars/MetaHuman/urdf/avatar_bulletworld.urdf.xacro (robot description, xacro)
@@ -118,24 +118,30 @@
         <xacro:default_inertial mass="5.50"/>
     </link>
+    <xacro:yaw_pitch_joints linkname="thigh_l" mass="5.50"/>
     <link name="${avatar_prefix}calf_l">
         <xacro:mesh_coll bpart="calf_l"/>
         <xacro:default_inertial mass="3.37"/>
     </link>
+     <xacro:yaw_pitch_joints linkname="calf_l" mass="3.37"/>
     <link name="${avatar_prefix}foot_l">
         <xacro:mesh_coll bpart="foot_l"/>
         <xacro:default_inertial mass="1.12"/>
     </link>
+    <xacro:yaw_pitch_joints linkname="foot_l" mass="1.12"/>
     <link name="${avatar_prefix}thigh_r">
         <xacro:mesh_coll bpart="thigh_r"/>
         <xacro:default_inertial mass="5.50"/>
     </link>
+    <xacro:yaw_pitch_joints linkname="thigh_r" mass="5.50"/>
     <link name="${avatar_prefix}calf_r">
         <xacro:mesh_coll bpart="calf_r"/>
         <xacro:default_inertial mass="3.37"/>
     </link>
+     <xacro:yaw_pitch_joints linkname="calf_r" mass="3.37"/>
     <link name="${avatar_prefix}foot_r">
         <xacro:mesh_coll bpart="foot_r"/>
         <xacro:default_inertial mass="1.12"/>
     </link>
+    <xacro:yaw_pitch_joints linkname="foot_r" mass="1.12"/>
     <joint name="${avatar_prefix}root_to_${avatar_prefix}pelvis_yaw" type="fixed">
         <parent link="${avatar_prefix}root"/>
@@ -165,7 +171,8 @@
         <axis xyz="1 0 0"/>
     </joint>
-    <joint name="${avatar_prefix}spine_01_to_${avatar_prefix}spine_02" type="continuous">
+    <joint name="${avatar_prefix}spine_01_to_${avatar_prefix}spine_02" type="revolute">
         <parent link="${avatar_prefix}spine_01"/>
         <child link="${avatar_prefix}spine_02"/>
+        <limit effort="1" lower="0" upper="0" velocity="1"/>
         <dynamics damping="1.0" friction="0.0001"/>
         <origin rpy="0 0 0" xyz="0.042 0 0"/>
@@ -200,8 +207,9 @@
         <axis xyz="1 0 0"/>
     </joint>
-    <joint name="${avatar_prefix}spine_04_to_${avatar_prefix}spine_05" type="continuous">
+    <joint name="${avatar_prefix}spine_04_to_${avatar_prefix}spine_05" type="revolute">
         <parent link="${avatar_prefix}spine_04"/>
         <child link="${avatar_prefix}spine_05"/>
         <dynamics damping="1.0" friction="0.0001"/>
+        <limit effort="1" lower="0" upper="0" velocity="1"/>
         <origin rpy="0 0 0" xyz="0.15038425 0 0"/>
         <axis xyz="1 0 0"/>
@@ -275,8 +283,9 @@
         <axis xyz="1 0 0"/>
     </joint>
-    <joint name="${avatar_prefix}upperarm_l_to_${avatar_prefix}lowerarm_l_yaw" type="continuous">
+    <joint name="${avatar_prefix}upperarm_l_to_${avatar_prefix}lowerarm_l_yaw" type="revolute">
         <parent link="${avatar_prefix}upperarm_l"/>
         <child link="${avatar_prefix}lowerarm_l_yaw"/>
         <origin rpy="0 0 0" xyz="0.238537997 0 0"/>
+        <limit effort="1" lower="-1.5708" upper="2.44346" velocity="1"/>
         <axis xyz="1 0 0"/>
     </joint>
@@ -295,8 +304,9 @@
         <axis xyz="1 0 0"/>
     </joint>
-    <joint name="${avatar_prefix}lowerarm_l_to_${avatar_prefix}hand_l_yaw" type="continuous">
+    <joint name="${avatar_prefix}lowerarm_l_to_${avatar_prefix}hand_l_yaw" type="revolute">
         <parent link="${avatar_prefix}lowerarm_l"/>
         <child link="${avatar_prefix}hand_l_yaw"/>
         <dynamics damping="1.0" friction="0.0001"/>
+        <limit effort="1" lower="0" upper="0" velocity="1"/>
         <origin rpy="-1.2351 0.1883 -0.2033" xyz="0.22966 0 -0.0000001"/>
         <axis xyz="1 0 0"/>
@@ -316,15 +326,17 @@
         <axis xyz="1 0 0"/>
     </joint>
-    <joint name="${avatar_prefix}spine_05_to_${avatar_prefix}clavicle_r" type="continuous">
+    <joint name="${avatar_prefix}spine_05_to_${avatar_prefix}clavicle_r" type="revolute">
         <parent link="${avatar_prefix}spine_05"/>
         <child link="${avatar_prefix}clavicle_r"/>
         <dynamics damping="1.0" friction="0.0001"/>
+        <limit effort="1" lower="0" upper="0" velocity="1"/>
         <origin rpy="3.14159 1.5708 0" xyz="0.05142808 0.00883206 0.00816548"/>
         <axis xyz="1 0 0"/>
     </joint>
-    <joint name="${avatar_prefix}clavicle_r_to_${avatar_prefix}upperarm_r_yaw" type="continuous">
+    <joint name="${avatar_prefix}clavicle_r_to_${avatar_prefix}upperarm_r_yaw" type="revolute">
         <parent link="${avatar_prefix}clavicle_r"/>
         <child link="${avatar_prefix}upperarm_r_yaw"/>
         <dynamics damping="1.0" friction="0.0001"/>
+        <limit effort="1" lower="0" upper="0" velocity="1"/>
         <origin rpy="0 1.0471975511965976 0" xyz="-0.13340 0 0"/>
         <axis xyz="1 0 0"/>
@@ -367,8 +379,9 @@
         <axis xyz="1 0 0"/>
     </joint>
-    <joint name="${avatar_prefix}lowerarm_r_to_${avatar_prefix}hand_r" type="continuous">
+    <joint name="${avatar_prefix}lowerarm_r_to_${avatar_prefix}hand_r_yaw" type="revolute">
         <parent link="${avatar_prefix}lowerarm_r"/>
         <child link="${avatar_prefix}hand_r_yaw"/>
         <dynamics damping="1.0" friction="0.0001"/>
+        <limit effort="1" lower="0" upper="0" velocity="1"/>
         <origin rpy="-1.2351 0.1883 -0.2033" xyz="-0.22 0 0"/>
         <axis xyz="1 0 0"/>
@@ -388,44 +401,134 @@
         <axis xyz="1 0 0"/>
     </joint>
-    <joint name="${avatar_prefix}pelvis_to_${avatar_prefix}thigh_l" type="continuous">
+    <joint name="${avatar_prefix}pelvis_to_${avatar_prefix}thigh_l_yaw" type="revolute">
         <parent link="${avatar_prefix}pelvis"/>
+        <child link="${avatar_prefix}thigh_l_yaw"/>
+        <dynamics damping="1.0" friction="0.0001"/>
+        <limit effort="1" lower="0" upper="0" velocity="1"/>
+        <origin rpy="0 0 0" xyz="-0.03036 0.003211013 -0.0957 "/>
+        <axis xyz="1 0 0"/>
+    </joint>
+     <joint name="${avatar_prefix}thigh_l_yaw_to_${avatar_prefix}thigh_l_pitch" type="revolute">
+        <parent link="${avatar_prefix}thigh_l_yaw"/>
+        <child link="${avatar_prefix}thigh_l_pitch"/>
+        <limit effort="1" lower="-1.5708" upper="2.44346" velocity="1"/>
+        <origin rpy="0 0 0" xyz="0 0 0"/>
+        <axis xyz="0 1 0"/>
+    </joint>
+    <joint name="${avatar_prefix}thigh_l_pitch_to_${avatar_prefix}thigh_l" type="revolute">
+        <parent link="${avatar_prefix}thigh_l_pitch"/>
         <child link="${avatar_prefix}thigh_l"/>
-        <dynamics damping="1.0" friction="0.0001"/>
-        <origin rpy="0 0 0" xyz="-0.03036 0.003211013 -0.0957 "/>
-        <axis xyz="1 0 0"/>
-    </joint>
-    <joint name="${avatar_prefix}thigh_l_to_${avatar_prefix}calf_l" type="continuous">
+        <limit effort="1" lower="-1.5708" upper="2.44346" velocity="1"/>
+        <origin rpy="0 0 0" xyz="0 0 0"/>
+        <axis xyz="1 0 0"/>
+    </joint>
+    <joint name="${avatar_prefix}thigh_l_to_${avatar_prefix}calf_l_yaw" type="revolute">
         <parent link="${avatar_prefix}thigh_l"/>
+        <child link="${avatar_prefix}calf_l_yaw"/>
+        <dynamics damping="1.0" friction="0.0001"/>
+        <limit effort="1" lower="0" upper="0" velocity="1"/>
+        <origin rpy="0 0 0" xyz="-0.4024 0 0"/>
+        <axis xyz="1 0 0"/>
+    </joint>
+     <joint name="${avatar_prefix}calf_l_yaw_to_${avatar_prefix}calf_l_pitch" type="revolute">
+        <parent link="${avatar_prefix}calf_l_yaw"/>
+        <child link="${avatar_prefix}calf_l_pitch"/>
+        <limit effort="1" lower="-1.5708" upper="2.44346" velocity="1"/>
+        <origin rpy="0 0 0" xyz="0 0 0"/>
+        <axis xyz="0 1 0"/>
+    </joint>
+    <joint name="${avatar_prefix}calf_l_pitch_to_${avatar_prefix}calf_l" type="revolute">
+        <parent link="${avatar_prefix}calf_l_pitch"/>
         <child link="${avatar_prefix}calf_l"/>
-        <dynamics damping="1.0" friction="0.0001"/>
-        <origin rpy="0 0 0" xyz="-0.4024 0 0"/>
-        <axis xyz="1 0 0"/>
-    </joint>
-    <joint name="${avatar_prefix}calf_l_to_${avatar_prefix}foot_l" type="continuous">
+        <limit effort="1" lower="-1.5708" upper="2.44346" velocity="1"/>
+        <origin rpy="0 0 0" xyz="0 0 0"/>
+        <axis xyz="1 0 0"/>
+    </joint>
+    <joint name="${avatar_prefix}calf_l_to_${avatar_prefix}foot_l_yaw" type="revolute">
         <parent link="${avatar_prefix}calf_l"/>
+        <child link="${avatar_prefix}foot_l_yaw"/>
+        <dynamics damping="1.0" friction="0.0001"/>
+        <limit effort="1" lower="0" upper="0" velocity="1"/>
+        <origin rpy="0 0 0" xyz="-0.3674 0 0"/>
+        <axis xyz="1 0 0"/>
+    </joint>
+     <joint name="${avatar_prefix}foot_l_yaw_to_${avatar_prefix}foot_l_pitch" type="revolute">
+        <parent link="${avatar_prefix}foot_l_yaw"/>
+        <child link="${avatar_prefix}foot_l_pitch"/>
+        <limit effort="1" lower="-1.5708" upper="2.44346" velocity="1"/>
+        <origin rpy="0 0 0" xyz="0 0 0"/>
+        <axis xyz="0 1 0"/>
+    </joint>
+    <joint name="${avatar_prefix}foot_l_pitch_to_${avatar_prefix}foot_l" type="revolute">
+        <parent link="${avatar_prefix}foot_l_pitch"/>
         <child link="${avatar_prefix}foot_l"/>
-        <dynamics damping="1.0" friction="0.0001"/>
-        <origin rpy="0 0 0" xyz="-0.3674 0 0"/>
-        <axis xyz="1 0 0"/>
-    </joint>
-    <joint name="${avatar_prefix}pelvis_to_${avatar_prefix}thigh_r" type="continuous">
+        <limit effort="1" lower="-1.5708" upper="2.44346" velocity="1"/>
+        <origin rpy="0 0 0" xyz="0 0 0"/>
+        <axis xyz="1 0 0"/>
+    </joint>
+    <joint name="${avatar_prefix}pelvis_to_${avatar_prefix}thigh_r_yaw" type="revolute">
         <parent link="${avatar_prefix}pelvis"/>
+        <child link="${avatar_prefix}thigh_r_yaw"/>
+        <dynamics damping="1.0" friction="0.0001"/>
+        <limit effort="1" lower="0" upper="0" velocity="1"/>
+        <origin rpy="0 0 -3.14159" xyz="-0.03036254 0.00325813 0.09572073"/>
+        <axis xyz="1 0 0"/>
+    </joint>
+     <joint name="${avatar_prefix}thigh_r_yaw_to_${avatar_prefix}thigh_r_pitch" type="revolute">
+        <parent link="${avatar_prefix}thigh_r_yaw"/>
+        <child link="${avatar_prefix}thigh_r_pitch"/>
+        <limit effort="1" lower="-1.5708" upper="2.44346" velocity="1"/>
+        <origin rpy="0 0 0" xyz="0 0 0"/>
+        <axis xyz="0 1 0"/>
+    </joint>
+    <joint name="${avatar_prefix}thigh_r_pitch_to_${avatar_prefix}thigh_r" type="revolute">
+        <parent link="${avatar_prefix}thigh_r_pitch"/>
         <child link="${avatar_prefix}thigh_r"/>
-        <dynamics damping="1.0" friction="0.0001"/>
-        <origin rpy="0 0 -3.14159" xyz="-0.03036254 0.00325813 0.09572073"/>
-        <axis xyz="1 0 0"/>
-    </joint>
-    <joint name="${avatar_prefix}thigh_r_to_${avatar_prefix}calf_r" type="continuous">
+        <limit effort="1" lower="-1.5708" upper="2.44346" velocity="1"/>
+        <origin rpy="0 0 0" xyz="0 0 0"/>
+        <axis xyz="1 0 0"/>
+    </joint>
+    <joint name="${avatar_prefix}thigh_r_to_${avatar_prefix}calf_r_yaw" type="revolute">
         <parent link="${avatar_prefix}thigh_r"/>
+        <child link="${avatar_prefix}calf_r_yaw"/>
+        <dynamics damping="1.0" friction="0.0001"/>
+        <limit effort="1" lower="0" upper="0" velocity="1"/>
+        <origin rpy="0 0 0" xyz="0.40552611 0 0"/>
+        <axis xyz="1 0 0"/>
+    </joint>
+    <joint name="${avatar_prefix}calf_r_yaw_to_${avatar_prefix}calf_r_pitch" type="revolute">
+        <parent link="${avatar_prefix}calf_r_yaw"/>
+        <child link="${avatar_prefix}calf_r_pitch"/>
+        <limit effort="1" lower="-1.5708" upper="2.44346" velocity="1"/>
+        <origin rpy="0 0 0" xyz="0 0 0"/>
+        <axis xyz="0 1 0"/>
+    </joint>
+    <joint name="${avatar_prefix}calf_r_pitch_to_${avatar_prefix}calf_r" type="revolute">
+        <parent link="${avatar_prefix}calf_r_pitch"/>
         <child link="${avatar_prefix}calf_r"/>
-        <dynamics damping="1.0" friction="0.0001"/>
-        <origin rpy="0 0 0" xyz="0.40552611 0 0"/>
-        <axis xyz="1 0 0"/>
-    </joint>
-    <joint name="${avatar_prefix}calf_r_to_${avatar_prefix}foot_r" type="continuous">
+        <limit effort="1" lower="-1.5708" upper="2.44346" velocity="1"/>
+        <origin rpy="0 0 0" xyz="0 0 0"/>
+        <axis xyz="1 0 0"/>
+    </joint>
+    <joint name="${avatar_prefix}calf_r_to_${avatar_prefix}foot_r_yaw" type="revolute">
         <parent link="${avatar_prefix}calf_r"/>
+        <child link="${avatar_prefix}foot_r_yaw"/>
+        <dynamics damping="1.0" friction="0.0001"/>
+        <limit effort="1" lower="0" upper="0" velocity="1"/>
+        <origin rpy="0 0 0" xyz="0.3674 0 0"/>
+        <axis xyz="1 0 0"/>
+    </joint>
+    <joint name="${avatar_prefix}foot_r_yaw_to_${avatar_prefix}foot_r_pitch" type="revolute">
+        <parent link="${avatar_prefix}foot_r_yaw"/>
+        <child link="${avatar_prefix}foot_r_pitch"/>
+        <limit effort="1" lower="-1.5708" upper="2.44346" velocity="1"/>
+        <origin rpy="0 0 0" xyz="0 0 0"/>
+        <axis xyz="0 1 0"/>
+    </joint>
+    <joint name="${avatar_prefix}foot_r_pitch_to_${avatar_prefix}foot_r" type="revolute">
+        <parent link="${avatar_prefix}foot_r_pitch"/>
         <child link="${avatar_prefix}foot_r"/>
-        <dynamics damping="1.0" friction="0.0001"/>
-        <origin rpy="0 0 0" xyz="0.3674 0 0"/>
+        <limit effort="1" lower="-1.5708" upper="2.44346" velocity="1"/>
+        <origin rpy="0 0 0" xyz="0 0 0"/>
         <axis xyz="1 0 0"/>
     </joint>
