Commit message: new joints for legs

File: avatars/MetaHuman/urdf/avatar_unrealengine.urdf.xacro (robot description, xacro)
@@ -15,10 +15,10 @@
         <visual>
             <geometry>
-                <mesh filename="${mesh_folder}/${bpart}.fbx" />
+                <mesh filename="${mesh_folder}/${bpart}.fbx"/>
             </geometry>
         </visual>
         <collision>
             <geometry>
-                <mesh filename="${mesh_folder}/${bpart}.fbx" />
+                <mesh filename="${mesh_folder}/${bpart}.fbx"/>
             </geometry>
         </collision>
@@ -106,24 +106,30 @@
         <xacro:default_inertial mass="5.50"/>
     </link>
+    <xacro:yaw_pitch_joints linkname="thigh_l" mass="5.50"/>
     <link name="${avatar_prefix}calf_l">
         <xacro:mesh_coll bpart="calf_l"/>
         <xacro:default_inertial mass="3.37"/>
     </link>
+     <xacro:yaw_pitch_joints linkname="calf_l" mass="3.37"/>
     <link name="${avatar_prefix}foot_l">
         <xacro:mesh_coll bpart="foot_l"/>
         <xacro:default_inertial mass="1.12"/>
     </link>
+    <xacro:yaw_pitch_joints linkname="foot_l" mass="1.12"/>
     <link name="${avatar_prefix}thigh_r">
         <xacro:mesh_coll bpart="thigh_r"/>
         <xacro:default_inertial mass="5.50"/>
     </link>
+    <xacro:yaw_pitch_joints linkname="thigh_r" mass="5.50"/>
     <link name="${avatar_prefix}calf_r">
         <xacro:mesh_coll bpart="calf_r"/>
         <xacro:default_inertial mass="3.37"/>
     </link>
+     <xacro:yaw_pitch_joints linkname="calf_r" mass="3.37"/>
     <link name="${avatar_prefix}foot_r">
         <xacro:mesh_coll bpart="foot_r"/>
         <xacro:default_inertial mass="1.12"/>
     </link>
+    <xacro:yaw_pitch_joints linkname="foot_r" mass="1.12"/>
     <joint name="${avatar_prefix}root_to_${avatar_prefix}pelvis_yaw" type="fixed">
         <parent link="${avatar_prefix}root"/>
@@ -153,7 +159,8 @@
         <axis xyz="1 0 0"/>
     </joint>
-    <joint name="${avatar_prefix}spine_01_to_${avatar_prefix}spine_02" type="continuous">
+    <joint name="${avatar_prefix}spine_01_to_${avatar_prefix}spine_02" type="revolute">
         <parent link="${avatar_prefix}spine_01"/>
         <child link="${avatar_prefix}spine_02"/>
+        <limit effort="1" lower="0" upper="0" velocity="1"/>
         <dynamics damping="1.0" friction="0.0001"/>
         <origin rpy="0 0 0" xyz="0.042 0 0"/>
@@ -188,8 +195,9 @@
         <axis xyz="1 0 0"/>
     </joint>
-    <joint name="${avatar_prefix}spine_04_to_${avatar_prefix}spine_05" type="continuous">
+    <joint name="${avatar_prefix}spine_04_to_${avatar_prefix}spine_05" type="revolute">
         <parent link="${avatar_prefix}spine_04"/>
         <child link="${avatar_prefix}spine_05"/>
         <dynamics damping="1.0" friction="0.0001"/>
+        <limit effort="1" lower="0" upper="0" velocity="1"/>
         <origin rpy="0 0 0" xyz="0.15038425 0 0"/>
         <axis xyz="1 0 0"/>
@@ -263,8 +271,9 @@
         <axis xyz="1 0 0"/>
     </joint>
-    <joint name="${avatar_prefix}upperarm_l_to_${avatar_prefix}lowerarm_l_yaw" type="continuous">
+    <joint name="${avatar_prefix}upperarm_l_to_${avatar_prefix}lowerarm_l_yaw" type="revolute">
         <parent link="${avatar_prefix}upperarm_l"/>
         <child link="${avatar_prefix}lowerarm_l_yaw"/>
         <origin rpy="0 0 0" xyz="0.238537997 0 0"/>
+        <limit effort="1" lower="-1.5708" upper="2.44346" velocity="1"/>
         <axis xyz="1 0 0"/>
     </joint>
@@ -283,8 +292,9 @@
         <axis xyz="1 0 0"/>
     </joint>
-    <joint name="${avatar_prefix}lowerarm_l_to_${avatar_prefix}hand_l_yaw" type="continuous">
+    <joint name="${avatar_prefix}lowerarm_l_to_${avatar_prefix}hand_l_yaw" type="revolute">
         <parent link="${avatar_prefix}lowerarm_l"/>
         <child link="${avatar_prefix}hand_l_yaw"/>
         <dynamics damping="1.0" friction="0.0001"/>
+        <limit effort="1" lower="0" upper="0" velocity="1"/>
         <origin rpy="-1.2351 0.1883 -0.2033" xyz="0.22966 0 -0.0000001"/>
         <axis xyz="1 0 0"/>
@@ -304,15 +314,17 @@
         <axis xyz="1 0 0"/>
     </joint>
-    <joint name="${avatar_prefix}spine_05_to_${avatar_prefix}clavicle_r" type="continuous">
+    <joint name="${avatar_prefix}spine_05_to_${avatar_prefix}clavicle_r" type="revolute">
         <parent link="${avatar_prefix}spine_05"/>
         <child link="${avatar_prefix}clavicle_r"/>
         <dynamics damping="1.0" friction="0.0001"/>
+        <limit effort="1" lower="0" upper="0" velocity="1"/>
         <origin rpy="3.14159 1.5708 0" xyz="0.05142808 0.00883206 0.00816548"/>
         <axis xyz="1 0 0"/>
     </joint>
-    <joint name="${avatar_prefix}clavicle_r_to_${avatar_prefix}upperarm_r_yaw" type="continuous">
+    <joint name="${avatar_prefix}clavicle_r_to_${avatar_prefix}upperarm_r_yaw" type="revolute">
         <parent link="${avatar_prefix}clavicle_r"/>
         <child link="${avatar_prefix}upperarm_r_yaw"/>
         <dynamics damping="1.0" friction="0.0001"/>
+        <limit effort="1" lower="0" upper="0" velocity="1"/>
         <origin rpy="0 1.0471975511965976 0" xyz="-0.13340 0 0"/>
         <axis xyz="1 0 0"/>
@@ -355,8 +367,9 @@
         <axis xyz="1 0 0"/>
     </joint>
-    <joint name="${avatar_prefix}lowerarm_r_to_${avatar_prefix}hand_r" type="continuous">
+    <joint name="${avatar_prefix}lowerarm_r_to_${avatar_prefix}hand_r_yaw" type="revolute">
         <parent link="${avatar_prefix}lowerarm_r"/>
         <child link="${avatar_prefix}hand_r_yaw"/>
         <dynamics damping="1.0" friction="0.0001"/>
+        <limit effort="1" lower="0" upper="0" velocity="1"/>
         <origin rpy="-1.2351 0.1883 -0.2033" xyz="-0.22 0 0"/>
         <axis xyz="1 0 0"/>
@@ -376,44 +389,134 @@
         <axis xyz="1 0 0"/>
     </joint>
-    <joint name="${avatar_prefix}pelvis_to_${avatar_prefix}thigh_l" type="continuous">
+    <joint name="${avatar_prefix}pelvis_to_${avatar_prefix}thigh_l_yaw" type="revolute">
         <parent link="${avatar_prefix}pelvis"/>
+        <child link="${avatar_prefix}thigh_l_yaw"/>
+        <dynamics damping="1.0" friction="0.0001"/>
+        <limit effort="1" lower="0" upper="0" velocity="1"/>
+        <origin rpy="0 0 0" xyz="-0.03036 0.003211013 -0.0957 "/>
+        <axis xyz="1 0 0"/>
+    </joint>
+     <joint name="${avatar_prefix}thigh_l_yaw_to_${avatar_prefix}thigh_l_pitch" type="revolute">
+        <parent link="${avatar_prefix}thigh_l_yaw"/>
+        <child link="${avatar_prefix}thigh_l_pitch"/>
+        <limit effort="1" lower="-1.5708" upper="2.44346" velocity="1"/>
+        <origin rpy="0 0 0" xyz="0 0 0"/>
+        <axis xyz="0 1 0"/>
+    </joint>
+    <joint name="${avatar_prefix}thigh_l_pitch_to_${avatar_prefix}thigh_l" type="revolute">
+        <parent link="${avatar_prefix}thigh_l_pitch"/>
         <child link="${avatar_prefix}thigh_l"/>
-        <dynamics damping="1.0" friction="0.0001"/>
-        <origin rpy="0 0 0" xyz="-0.03036 0.003211013 -0.0957 "/>
-        <axis xyz="1 0 0"/>
-    </joint>
-    <joint name="${avatar_prefix}thigh_l_to_${avatar_prefix}calf_l" type="continuous">
+        <limit effort="1" lower="-1.5708" upper="2.44346" velocity="1"/>
+        <origin rpy="0 0 0" xyz="0 0 0"/>
+        <axis xyz="1 0 0"/>
+    </joint>
+    <joint name="${avatar_prefix}thigh_l_to_${avatar_prefix}calf_l_yaw" type="revolute">
         <parent link="${avatar_prefix}thigh_l"/>
+        <child link="${avatar_prefix}calf_l_yaw"/>
+        <dynamics damping="1.0" friction="0.0001"/>
+        <limit effort="1" lower="0" upper="0" velocity="1"/>
+        <origin rpy="0 0 0" xyz="-0.4024 0 0"/>
+        <axis xyz="1 0 0"/>
+    </joint>
+     <joint name="${avatar_prefix}calf_l_yaw_to_${avatar_prefix}calf_l_pitch" type="revolute">
+        <parent link="${avatar_prefix}calf_l_yaw"/>
+        <child link="${avatar_prefix}calf_l_pitch"/>
+        <limit effort="1" lower="-1.5708" upper="2.44346" velocity="1"/>
+        <origin rpy="0 0 0" xyz="0 0 0"/>
+        <axis xyz="0 1 0"/>
+    </joint>
+    <joint name="${avatar_prefix}calf_l_pitch_to_${avatar_prefix}calf_l" type="revolute">
+        <parent link="${avatar_prefix}calf_l_pitch"/>
         <child link="${avatar_prefix}calf_l"/>
-        <dynamics damping="1.0" friction="0.0001"/>
-        <origin rpy="0 0 0" xyz="-0.4024 0 0"/>
-        <axis xyz="1 0 0"/>
-    </joint>
-    <joint name="${avatar_prefix}calf_l_to_${avatar_prefix}foot_l" type="continuous">
+        <limit effort="1" lower="-1.5708" upper="2.44346" velocity="1"/>
+        <origin rpy="0 0 0" xyz="0 0 0"/>
+        <axis xyz="1 0 0"/>
+    </joint>
+    <joint name="${avatar_prefix}calf_l_to_${avatar_prefix}foot_l_yaw" type="revolute">
         <parent link="${avatar_prefix}calf_l"/>
+        <child link="${avatar_prefix}foot_l_yaw"/>
+        <dynamics damping="1.0" friction="0.0001"/>
+        <limit effort="1" lower="0" upper="0" velocity="1"/>
+        <origin rpy="0 0 0" xyz="-0.3674 0 0"/>
+        <axis xyz="1 0 0"/>
+    </joint>
+     <joint name="${avatar_prefix}foot_l_yaw_to_${avatar_prefix}foot_l_pitch" type="revolute">
+        <parent link="${avatar_prefix}foot_l_yaw"/>
+        <child link="${avatar_prefix}foot_l_pitch"/>
+        <limit effort="1" lower="-1.5708" upper="2.44346" velocity="1"/>
+        <origin rpy="0 0 0" xyz="0 0 0"/>
+        <axis xyz="0 1 0"/>
+    </joint>
+    <joint name="${avatar_prefix}foot_l_pitch_to_${avatar_prefix}foot_l" type="revolute">
+        <parent link="${avatar_prefix}foot_l_pitch"/>
         <child link="${avatar_prefix}foot_l"/>
-        <dynamics damping="1.0" friction="0.0001"/>
-        <origin rpy="0 0 0" xyz="-0.3674 0 0"/>
-        <axis xyz="1 0 0"/>
-    </joint>
-    <joint name="${avatar_prefix}pelvis_to_${avatar_prefix}thigh_r" type="continuous">
+        <limit effort="1" lower="-1.5708" upper="2.44346" velocity="1"/>
+        <origin rpy="0 0 0" xyz="0 0 0"/>
+        <axis xyz="1 0 0"/>
+    </joint>
+    <joint name="${avatar_prefix}pelvis_to_${avatar_prefix}thigh_r_yaw" type="revolute">
         <parent link="${avatar_prefix}pelvis"/>
+        <child link="${avatar_prefix}thigh_r_yaw"/>
+        <dynamics damping="1.0" friction="0.0001"/>
+        <limit effort="1" lower="0" upper="0" velocity="1"/>
+        <origin rpy="0 0 -3.14159" xyz="-0.03036254 0.00325813 0.09572073"/>
+        <axis xyz="1 0 0"/>
+    </joint>
+     <joint name="${avatar_prefix}thigh_r_yaw_to_${avatar_prefix}thigh_r_pitch" type="revolute">
+        <parent link="${avatar_prefix}thigh_r_yaw"/>
+        <child link="${avatar_prefix}thigh_r_pitch"/>
+        <limit effort="1" lower="-1.5708" upper="2.44346" velocity="1"/>
+        <origin rpy="0 0 0" xyz="0 0 0"/>
+        <axis xyz="0 1 0"/>
+    </joint>
+    <joint name="${avatar_prefix}thigh_r_pitch_to_${avatar_prefix}thigh_r" type="revolute">
+        <parent link="${avatar_prefix}thigh_r_pitch"/>
         <child link="${avatar_prefix}thigh_r"/>
-        <dynamics damping="1.0" friction="0.0001"/>
-        <origin rpy="0 0 -3.14159" xyz="-0.03036254 0.00325813 0.09572073"/>
-        <axis xyz="1 0 0"/>
-    </joint>
-    <joint name="${avatar_prefix}thigh_r_to_${avatar_prefix}calf_r" type="continuous">
+        <limit effort="1" lower="-1.5708" upper="2.44346" velocity="1"/>
+        <origin rpy="0 0 0" xyz="0 0 0"/>
+        <axis xyz="1 0 0"/>
+    </joint>
+    <joint name="${avatar_prefix}thigh_r_to_${avatar_prefix}calf_r_yaw" type="revolute">
         <parent link="${avatar_prefix}thigh_r"/>
+        <child link="${avatar_prefix}calf_r_yaw"/>
+        <dynamics damping="1.0" friction="0.0001"/>
+        <limit effort="1" lower="0" upper="0" velocity="1"/>
+        <origin rpy="0 0 0" xyz="0.40552611 0 0"/>
+        <axis xyz="1 0 0"/>
+    </joint>
+    <joint name="${avatar_prefix}calf_r_yaw_to_${avatar_prefix}calf_r_pitch" type="revolute">
+        <parent link="${avatar_prefix}calf_r_yaw"/>
+        <child link="${avatar_prefix}calf_r_pitch"/>
+        <limit effort="1" lower="-1.5708" upper="2.44346" velocity="1"/>
+        <origin rpy="0 0 0" xyz="0 0 0"/>
+        <axis xyz="0 1 0"/>
+    </joint>
+    <joint name="${avatar_prefix}calf_r_pitch_to_${avatar_prefix}calf_r" type="revolute">
+        <parent link="${avatar_prefix}calf_r_pitch"/>
         <child link="${avatar_prefix}calf_r"/>
-        <dynamics damping="1.0" friction="0.0001"/>
-        <origin rpy="0 0 0" xyz="0.40552611 0 0"/>
-        <axis xyz="1 0 0"/>
-    </joint>
-    <joint name="${avatar_prefix}calf_r_to_${avatar_prefix}foot_r" type="continuous">
+        <limit effort="1" lower="-1.5708" upper="2.44346" velocity="1"/>
+        <origin rpy="0 0 0" xyz="0 0 0"/>
+        <axis xyz="1 0 0"/>
+    </joint>
+    <joint name="${avatar_prefix}calf_r_to_${avatar_prefix}foot_r_yaw" type="revolute">
         <parent link="${avatar_prefix}calf_r"/>
+        <child link="${avatar_prefix}foot_r_yaw"/>
+        <dynamics damping="1.0" friction="0.0001"/>
+        <limit effort="1" lower="0" upper="0" velocity="1"/>
+        <origin rpy="0 0 0" xyz="0.3674 0 0"/>
+        <axis xyz="1 0 0"/>
+    </joint>
+    <joint name="${avatar_prefix}foot_r_yaw_to_${avatar_prefix}foot_r_pitch" type="revolute">
+        <parent link="${avatar_prefix}foot_r_yaw"/>
+        <child link="${avatar_prefix}foot_r_pitch"/>
+        <limit effort="1" lower="-1.5708" upper="2.44346" velocity="1"/>
+        <origin rpy="0 0 0" xyz="0 0 0"/>
+        <axis xyz="0 1 0"/>
+    </joint>
+    <joint name="${avatar_prefix}foot_r_pitch_to_${avatar_prefix}foot_r" type="revolute">
+        <parent link="${avatar_prefix}foot_r_pitch"/>
         <child link="${avatar_prefix}foot_r"/>
-        <dynamics damping="1.0" friction="0.0001"/>
-        <origin rpy="0 0 0" xyz="0.3674 0 0"/>
+        <limit effort="1" lower="-1.5708" upper="2.44346" velocity="1"/>
+        <origin rpy="0 0 0" xyz="0 0 0"/>
         <axis xyz="1 0 0"/>
     </joint>

Commit message: changed to ue model

File: avatars/MetaHuman/urdf/avatar_bulletworld.urdf.xacro (robot description, xacro)
@@ -191,5 +191,5 @@
         <limit effort="1" lower="0" upper="0" velocity="1"/>
         <origin rpy="0 0 0" xyz="0.07891 0 0"/>
-        <axis xyz="1 0 0"/>
+        <axis xyz="0 0 1"/>
     </joint>
     <joint name="${avatar_prefix}spine_04_yaw_to_${avatar_prefix}spine_04_pitch" type="revolute">
@@ -237,5 +237,5 @@
         <limit effort="1" lower="-0.610865" upper="0.610865" velocity="1"/>
         <origin rpy="0 0 0" xyz="0.05279524 0 0"/>
-        <axis xyz="0 1 0"/>
+        <axis xyz="0 0 1"/>
     </joint>
     <joint name="${avatar_prefix}head_yaw_to_${avatar_prefix}head_pitch" type="revolute">
@@ -288,5 +288,5 @@
         <origin rpy="0 0 0" xyz="0.238537997 0 0"/>
         <limit effort="1" lower="-1.5708" upper="2.44346" velocity="1"/>
-        <axis xyz="1 0 0"/>
+        <axis xyz="0 0 1"/>
     </joint>
     <joint name="${avatar_prefix}lowerarm_l_yaw_to_${avatar_prefix}lowerarm_l_pitch" type="revolute">
@@ -310,5 +310,5 @@
         <limit effort="1" lower="0" upper="0" velocity="1"/>
         <origin rpy="-1.2351 0.1883 -0.2033" xyz="0.22966 0 -0.0000001"/>
-        <axis xyz="1 0 0"/>
+        <axis xyz="0 0 1"/>
     </joint>
     <joint name="${avatar_prefix}hand_l_yaw_to_${avatar_prefix}hand_l_pitch" type="revolute">
@@ -340,5 +340,5 @@
         <limit effort="1" lower="0" upper="0" velocity="1"/>
         <origin rpy="0 1.0471975511965976 0" xyz="-0.13340 0 0"/>
-        <axis xyz="1 0 0"/>
+        <axis xyz="0 0 1"/>
     </joint>
     <joint name="${avatar_prefix}upperarm_r_yaw_to_${avatar_prefix}upperarm_r_pitch" type="revolute">
@@ -363,5 +363,5 @@
         <dynamics damping="1.0" friction="0.0001"/>
         <origin rpy="0 0 0" xyz="-0.2383 0 0"/>
-        <axis xyz="1 0 0"/>
+        <axis xyz="0 0 1"/>
     </joint>
     <joint name="${avatar_prefix}lowerarm_r_yaw_to_${avatar_prefix}lowerarm_r_pitch" type="revolute">
@@ -385,5 +385,5 @@
         <limit effort="1" lower="0" upper="0" velocity="1"/>
         <origin rpy="-1.2351 0.1883 -0.2033" xyz="-0.22 0 0"/>
-        <axis xyz="1 0 0"/>
+        <axis xyz="0 0 1"/>
     </joint>
     <joint name="${avatar_prefix}hand_r_yaw_to_${avatar_prefix}hand_r_pitch" type="revolute">
@@ -405,12 +405,12 @@
         <child link="${avatar_prefix}thigh_l_yaw"/>
         <dynamics damping="1.0" friction="0.0001"/>
-        <limit effort="1" lower="0" upper="0" velocity="1"/>
+        <limit effort="1" lower="-1.5708" upper="2.44346" velocity="1"/>
         <origin rpy="0 0 0" xyz="-0.03036 0.003211013 -0.0957 "/>
-        <axis xyz="1 0 0"/>
+        <axis xyz="0 0 1"/>
     </joint>
      <joint name="${avatar_prefix}thigh_l_yaw_to_${avatar_prefix}thigh_l_pitch" type="revolute">
         <parent link="${avatar_prefix}thigh_l_yaw"/>
         <child link="${avatar_prefix}thigh_l_pitch"/>
-        <limit effort="1" lower="-1.5708" upper="2.44346" velocity="1"/>
+        <limit effort="1" lower="-0.52" upper="0.87" velocity="1"/>
         <origin rpy="0 0 0" xyz="0 0 0"/>
         <axis xyz="0 1 0"/>
@@ -423,9 +423,10 @@
         <axis xyz="1 0 0"/>
     </joint>
+     <!-- left knee extension/flexion-->
     <joint name="${avatar_prefix}thigh_l_to_${avatar_prefix}calf_l_yaw" type="revolute">
         <parent link="${avatar_prefix}thigh_l"/>
         <child link="${avatar_prefix}calf_l_yaw"/>
         <dynamics damping="1.0" friction="0.0001"/>
-        <limit effort="1" lower="0" upper="0" velocity="1"/>
+        <limit effort="1" lower="0" upper="2.61799" velocity="1"/>
         <origin rpy="0 0 0" xyz="-0.4024 0 0"/>
         <axis xyz="1 0 0"/>
@@ -434,5 +435,5 @@
         <parent link="${avatar_prefix}calf_l_yaw"/>
         <child link="${avatar_prefix}calf_l_pitch"/>
-        <limit effort="1" lower="-1.5708" upper="2.44346" velocity="1"/>
+        <limit effort="1" lower="0" upper="0" velocity="1"/>
         <origin rpy="0 0 0" xyz="0 0 0"/>
         <axis xyz="0 1 0"/>
@@ -441,5 +442,5 @@
         <parent link="${avatar_prefix}calf_l_pitch"/>
         <child link="${avatar_prefix}calf_l"/>
-        <limit effort="1" lower="-1.5708" upper="2.44346" velocity="1"/>
+        <limit effort="1" lower="0" upper="0" velocity="1"/>
         <origin rpy="0 0 0" xyz="0 0 0"/>
         <axis xyz="1 0 0"/>
@@ -451,5 +452,5 @@
         <limit effort="1" lower="0" upper="0" velocity="1"/>
         <origin rpy="0 0 0" xyz="-0.3674 0 0"/>
-        <axis xyz="1 0 0"/>
+        <axis xyz="0 0 1"/>
     </joint>
      <joint name="${avatar_prefix}foot_l_yaw_to_${avatar_prefix}foot_l_pitch" type="revolute">
@@ -473,10 +474,10 @@
         <limit effort="1" lower="0" upper="0" velocity="1"/>
         <origin rpy="0 0 -3.14159" xyz="-0.03036254 0.00325813 0.09572073"/>
-        <axis xyz="1 0 0"/>
+        <axis xyz="0 0 1"/>
     </joint>
      <joint name="${avatar_prefix}thigh_r_yaw_to_${avatar_prefix}thigh_r_pitch" type="revolute">
         <parent link="${avatar_prefix}thigh_r_yaw"/>
         <child link="${avatar_prefix}thigh_r_pitch"/>
-        <limit effort="1" lower="-1.5708" upper="2.44346" velocity="1"/>
+        <limit effort="1" lower="-0.52" upper="0.87" velocity="1"/>
         <origin rpy="0 0 0" xyz="0 0 0"/>
         <axis xyz="0 1 0"/>
@@ -495,5 +496,5 @@
         <limit effort="1" lower="0" upper="0" velocity="1"/>
         <origin rpy="0 0 0" xyz="0.40552611 0 0"/>
-        <axis xyz="1 0 0"/>
+        <axis xyz="0 0 1"/>
     </joint>
     <joint name="${avatar_prefix}calf_r_yaw_to_${avatar_prefix}calf_r_pitch" type="revolute">
@@ -517,5 +518,5 @@
         <limit effort="1" lower="0" upper="0" velocity="1"/>
         <origin rpy="0 0 0" xyz="0.3674 0 0"/>
-        <axis xyz="1 0 0"/>
+        <axis xyz="0 0 1"/>
     </joint>
     <joint name="${avatar_prefix}foot_r_yaw_to_${avatar_prefix}foot_r_pitch" type="revolute">

Commit message: add camera_frame

File: avatars/MetaHuman/urdf/avatar_bulletworld.urdf.xacro (robot description, xacro)
@@ -534,3 +534,10 @@
         <axis xyz="1 0 0"/>
     </joint>
+    <!-- "Camera to see relative to root -->
+     <link name="Camera_frame_avatar"/>
+  <joint name="Camera_frame_avatar_fixedjoint" type="fixed">
+    <parent link="root"/>
+    <child link="Camera_frame_avatar"/>
+    <origin rpy="-1.57079632679 0 -1.57079632679" xyz="0.05138 0.039 1.4194"/>
+  </joint>
 </robot>
